File: pcb/ai_breakout_MCP4725.brd (EAGLE design)
At the start: 15.2 x 7.6 mm, 10 parts, among them J1 1X03, J2 1X03NOFIRST, U1 MCP4725

Commit message: gerber file created
Parts:
- U1: value MCP4725 -> MCP4725SOT-23
Other:
- board text added: "JCH v1.0"
- board text removed: "JCH_Ver.1.0"
Changed lines of the file:
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@@
 <setting verticaltext="up"/>
 </settings>
-<grid distance="5" unitdist="mil" unit="mil" style="lines" multiple="1" display="yes" altdistance="0.025" altunitdist="inch" altunit="inch"/>
+<grid distance="10" unitdist="mil" unit="mil" style="lines" multiple="1" display="yes" altdistance="0.025" altunitdist="inch" altunit="inch"/>
 <layers>
 <layer number="1" name="Top" color="4" fill="1" visible="yes" active="yes"/>
@@
 <wire x1="15.24" y1="7.62" x2="15.24" y2="0" width="0.0254" layer="20"/>
 <wire x1="15.24" y1="0" x2="0" y2="0" width="0.0254" layer="20"/>
-<text x="11.9126" y="4.5466" size="0.6096" layer="25" font="vector" rot="SR270">SDA</text>
-<text x="11.938" y="7.112" size="0.6096" layer="25" font="vector" rot="SR270">SCL</text>
-<text x="11.938" y="2.032" size="0.6096" layer="25" font="vector" rot="SR270">GND</text>
-<text x="3.302" y="0.508" size="0.6096" layer="25" font="vector" rot="R90">VDD</text>
-<text x="3.302" y="5.334" size="0.6096" layer="25" font="vector" rot="R90">VOUT</text>
-<text x="3.302" y="3.048" size="0.6096" layer="25" font="vector" rot="SR90">GND</text>
-<text x="11.43" y="5.588" size="0.6096" layer="26" font="vector" rot="MR0">Digital - Analog</text>
-<text x="9.398" y="4.826" size="0.6096" layer="26" font="vector" rot="MR0">Converter</text>
-<text x="11.684" y="3.048" size="0.6096" layer="26" font="vector" rot="MR0">www.acrobotic.com</text>
-<text x="12.573" y="0.127" size="0.3048" layer="26" font="fixed" rot="MR0">JCH_Ver.1.0</text>
-<text x="9.017" y="6.35" size="0.6096" layer="26" font="vector" rot="MR0">MCP4725</text>
+<text x="12.4206" y="3.0734" size="0.6096" layer="25" font="vector" ratio="10" rot="SR90">SDA</text>
+<text x="12.446" y="5.588" size="0.6096" layer="25" font="vector" ratio="10" rot="SR90">SCL</text>
+<text x="12.446" y="0.508" size="0.6096" layer="25" font="vector" ratio="10" rot="SR90">GND</text>
+<text x="2.794" y="2.032" size="0.6096" layer="25" font="vector" ratio="10" rot="SR270">VDD</text>
+<text x="2.794" y="7.366" size="0.6096" layer="25" font="vector" ratio="10" rot="SR270">VOUT</text>
+<text x="2.794" y="4.572" size="0.6096" layer="25" font="vector" ratio="10" rot="SR270">GND</text>
+<text x="11.43" y="5.588" size="0.6096" layer="26" font="vector" ratio="10" rot="MR0">Digital - Analog</text>
+<text x="9.398" y="4.826" size="0.6096" layer="26" font="vector" ratio="10" rot="MR0">Converter</text>
+<text x="11.684" y="3.048" size="0.6096" layer="26" font="vector" ratio="10" rot="MR0">www.acrobotic.com</text>
+<text x="12.573" y="0.127" size="0.3048" layer="26" font="fixed" rot="MR0">JCH v1.0</text>
+<text x="9.017" y="6.35" size="0.6096" layer="26" font="vector" ratio="10" rot="MR0">MCP4725</text>
 </plain>
 <attributes>
@@
 <attribute name="NAME" x="5.5118" y="6.0452" size="0.4064" layer="25" font="vector" ratio="10" rot="R180"/>
 </element>
-<element name="U1" library="Ai_IC" package="SOT23-6" value="MCP4725" x="7.747" y="4.3942" smashed="yes" rot="R270">
-<attribute name="PROD_ID" value="IC-08886" x="7.747" y="4.3942" size="1.778" layer="27" rot="R270" display="off"/>
+<element name="U1" library="Ai_IC" package="SOT23-6" value="MCP4725SOT-23" x="7.747" y="4.3942" smashed="yes" rot="R270">
 <attribute name="NAME" x="8.0518" y="2.8448" size="0.4064" layer="25" font="vector" ratio="10" rot="R180"/>
 </element>
